Commit message: tested urdf.xacro>urdf using command line, updated xacro file accordingly

File: nuturtle_description/urdf/turtle3.urdf (robot description, URDF)
Before this commit: robot turtlebot3_burger, 7 links, 6 joints
Links:
- link base_link: geometry collision box size=0.14200000000000002 0.14200000000000002 0.14200000000000002; visual mesh filename=package://meshes/burger_base.stl scale=0.001 0.001 0.001
- link wheel_left_link: geometry collision cylinder length=0.018 radius=0.033; visual mesh filename=package://meshes/left_tire.stl scale=0.001 0.001 0.001
- link wheel_right_link: geometry collision cylinder length=0.018 radius=0.033; visual mesh filename=package://meshes/right_tire.stl scale=0.001 0.001 0.001
Joints:
- joint wheel_left_joint: origin xyz=0.0 ${track_width/2} 0.023 rpy=-1.57 0 0 -> xyz=0.0 0.08 0.023 rpy=-1.57 0 0
- joint wheel_right_joint: origin xyz=0.0 ${track_width/(-2)} 0.023 rpy=-1.57 0 0 -> xyz=0.0 -0.08 0.023 rpy=-1.57 0 0
