Commit message: updated urdfxacro and cmakelists, package accordingly

File: nuturtle_description/urdf/turtlebot3_burger.urdf.xacro (robot description, xacro)
@@ -2,5 +2,5 @@
 <robot name="turtlebot3_burger"
   xmlns:xacro="http://ros.org/wiki/xacro">
-  <!-- <xacro:include filename="$(find turtlebot3_description)/urdf/common_properties.urdf"/> -->
+  <!-- <xacro:include filename="$(find nuturtle_description)/urdf/common_properties.urdf"/> -->
   <!-- Init colour -->
   <material name="black">
@@ -44,5 +44,5 @@
       <origin xyz="-0.032 0 0.0" rpy="0 0 0"/>
       <geometry>
-        <mesh filename="package://turtlebot3_description/meshes/bases/burger_base.stl" scale="0.001 0.001 0.001"/>
+        <mesh filename="package://meshes/burger_base.stl" scale="0.001 0.001 0.001"/>
       </geometry>
       <material name="light_black"/>
@@ -70,5 +70,5 @@
       <origin xyz="0 0 0" rpy="1.57 0 0"/>
       <geometry>
-        <mesh filename="package://turtlebot3_description/meshes/wheels/left_tire.stl" scale="0.001 0.001 0.001"/>
+        <mesh filename="package://meshes/left_tire.stl" scale="0.001 0.001 0.001"/>
       </geometry>
       <material name="dark"/>
@@ -96,5 +96,5 @@
       <origin xyz="0 0 0" rpy="1.57 0 0"/>
       <geometry>
-        <mesh filename="package://turtlebot3_description/meshes/wheels/right_tire.stl" scale="0.001 0.001 0.001"/>
+        <mesh filename="package://meshes/right_tire.stl" scale="0.001 0.001 0.001"/>
       </geometry>
       <material name="dark"/>
@@ -145,5 +145,5 @@
       <origin xyz="0 0 0.0" rpy="0 0 0"/>
       <geometry>
-        <mesh filename="package://turtlebot3_description/meshes/sensors/lds.stl" scale="0.001 0.001 0.001"/>
+        <mesh filename="package://meshes/lds.stl" scale="0.001 0.001 0.001"/>
       </geometry>
       <material name="dark"/>

Commit message: created yaml file for parameters and appropriate macros for xacro

File: nuturtle_description/urdf/turtlebot3_burger.urdf.xacro (robot description, xacro)
@@ -1,6 +1,12 @@
+<!--This file has been modified from the original version as per APLv2-->
 <?xml version="1.0" ?>
 <robot name="turtlebot3_burger"
   xmlns:xacro="http://ros.org/wiki/xacro">
   <!-- <xacro:include filename="$(find nuturtle_description)/urdf/common_properties.urdf"/> -->
+  <xacro:property name="yaml_file" value="$(find nuturtle_description)/config/diff_params.yaml" />
+  <xacro:property name="props" value="${load_yaml(yaml_file)['/**']['ros__parameters']}" />
+  <xacro:property name="wheel_radius" value="${props['wheel_radius']}" />
+  <xacro:property name="track_width" value="${props['track_width']}" />
+  <xacro:property name="collision_radius" value="${props['collision_radius']}"
   <!-- Init colour -->
   <material name="black">
@@ -51,5 +57,8 @@
       <origin xyz="-0.032 0 0.070" rpy="0 0 0"/>
       <geometry>
-        <box size="0.140 0.140 0.143"/>
+        <xacro:if value="${collision_radius &lt 0}">
+          <box size="0.140 0.140 0.143"/>
+        <xacro:if value="${collision_radius &gt 0}">
+          <box size="${0.032+collision_radius} ${0.032+collision_radius} ${0.032+collision_radius}">
       </geometry>
     </collision>
@@ -63,5 +72,5 @@
     <parent link="base_link"/>
     <child link="wheel_left_link"/>
-    <origin xyz="0.0 0.08 0.023" rpy="-1.57 0 0"/>
+    <origin xyz="0.0 ${track_width/2} 0.023" rpy="-1.57 0 0"/>
     <axis xyz="0 0 1"/>
   </joint>
@@ -77,5 +86,5 @@
       <origin xyz="0 0 0" rpy="0 0 0"/>
       <geometry>
-        <cylinder length="0.018" radius="0.033"/>
+        <cylinder length="0.018" radius="${wheel_radius}"/>
       </geometry>
     </collision>
@@ -89,5 +98,5 @@
     <parent link="base_link"/>
     <child link="wheel_right_link"/>
-    <origin xyz="0.0 -0.080 0.023" rpy="-1.57 0 0"/>
+    <origin xyz="0.0 ${track_width/(-2)} 0.023" rpy="-1.57 0 0"/>
     <axis xyz="0 0 1"/>
   </joint>
@@ -103,5 +112,5 @@
       <origin xyz="0 0 0" rpy="0 0 0"/>
       <geometry>
-        <cylinder length="0.018" radius="0.033"/>
+        <cylinder length="0.018" radius="${wheel_radius}"/>
       </geometry>
     </collision>

Commit message: fixed urdf find meshes error. saved rviz config. successful rviz build

File: nuturtle_description/urdf/turtlebot3_burger.urdf.xacro (robot description, xacro)
@@ -5,5 +5,5 @@
   <!-- <xacro:include filename="$(find nuturtle_description)/urdf/common_properties.urdf"/> -->
   <xacro:property name="yaml_file" value="$(find nuturtle_description)/config/diff_params.yaml" />
-  <xacro:property name="props" value="${load_yaml(yaml_file)['/**']['ros__parameters']}" />
+  <xacro:property name="props" value="${xacro.load_yaml(yaml_file)['/**']['ros__parameters']}" />
   <xacro:property name="wheel_radius" value="${props['wheel_radius']}" />
   <xacro:property name="track_width" value="${props['track_width']}" />
@@ -50,5 +50,5 @@
       <origin xyz="-0.032 0 0.0" rpy="0 0 0"/>
       <geometry>
-        <mesh filename="package://meshes/burger_base.stl" scale="0.001 0.001 0.001"/>
+        <mesh filename="package://nuturtle_description/meshes/burger_base.stl" scale="0.001 0.001 0.001"/>
       </geometry>
       <material name="light_black"/>
@@ -81,5 +81,5 @@
       <origin xyz="0 0 0" rpy="1.57 0 0"/>
       <geometry>
-        <mesh filename="package://meshes/left_tire.stl" scale="0.001 0.001 0.001"/>
+        <mesh filename="package://nuturtle_description/meshes/left_tire.stl" scale="0.001 0.001 0.001"/>
       </geometry>
       <material name="dark"/>
@@ -107,5 +107,5 @@
       <origin xyz="0 0 0" rpy="1.57 0 0"/>
       <geometry>
-        <mesh filename="package://meshes/right_tire.stl" scale="0.001 0.001 0.001"/>
+        <mesh filename="package://nuturtle_description/meshes/right_tire.stl" scale="0.001 0.001 0.001"/>
       </geometry>
       <material name="dark"/>
@@ -156,5 +156,5 @@
       <origin xyz="0 0 0.0" rpy="0 0 0"/>
       <geometry>
-        <mesh filename="package://meshes/lds.stl" scale="0.001 0.001 0.001"/>
+        <mesh filename="package://nuturtle_description/meshes/lds.stl" scale="0.001 0.001 0.001"/>
       </geometry>
       <material name="dark"/>

Commit message: created .gitignore file. modified xacro and launch file to pass color argument. deleted unneeded xacro file

File: nuturtle_description/urdf/turtlebot3_burger.urdf.xacro (robot description, xacro)
@@ -3,10 +3,10 @@
   xmlns:xacro="http://ros.org/wiki/xacro">
   <!--This file has been modified from the original version as per APLv2-->
-  <!-- <xacro:include filename="$(find nuturtle_description)/urdf/common_properties.urdf"/> -->
-  <xacro:property name="yaml_file" value="$(find nuturtle_description)/config/diff_params.yaml" />
-  <xacro:property name="props" value="${xacro.load_yaml(yaml_file)['/**']['ros__parameters']}" />
-  <xacro:property name="wheel_radius" value="${props['wheel_radius']}" />
-  <xacro:property name="track_width" value="${props['track_width']}" />
-  <xacro:property name="collision_radius" value="${props['collision_radius']}" />
+  <xacro:property name="yaml_file" value="$(find nuturtle_description)/config/diff_params.yaml" />  <!--loads parameter yaml file-->
+  <xacro:property name="props" value="${xacro.load_yaml(yaml_file)['/**']['ros__parameters']}" />   <!--loads parameters from yaml file-->
+  <xacro:property name="wheel_radius" value="${props['wheel_radius']}" />         <!--creates macro for wheel_radius parameter-->
+  <xacro:property name="track_width" value="${props['track_width']}" />           <!--creates macro for track_width parameter-->
+  <xacro:property name="collision_radius" value="${props['collision_radius']}" /> <!--creates macro for collision_radius parameter-->
+  <xacro:arg name="color" default="purple"/>                                      <!--takes in argument for color from launchfile-->
   <!-- Init colour -->
   <material name="black">
@@ -40,4 +40,7 @@
     <color rgba="1.0 1.0 1.0 1.0"/>
   </material>
+  <material name="purple">
+    <color rgba="0.3 0.16 0.52 1.0"/>
+  </material>
   <link name="base_footprint"/>
   <joint name="base_joint" type="fixed">
@@ -52,14 +55,14 @@
         <mesh filename="package://nuturtle_description/meshes/burger_base.stl" scale="0.001 0.001 0.001"/>
       </geometry>
-      <material name="light_black"/>
+      <material name="$(arg color)"/>
     </visual>
     <collision>
       <origin xyz="-0.032 0 0.070" rpy="0 0 0"/>
       <geometry>
-        <xacro:if value="${collision_radius &lt; 0}">
+        <xacro:if value="${collision_radius &lt; 0}">                                                 <!--If collision radius parameter is negative, use default value-->
           <box size="0.140 0.140 0.143"/>
         </xacro:if>
         <xacro:if value="${collision_radius &gt; 0}">
-          <box size="${0.032+collision_radius} ${0.032+collision_radius} ${0.032+collision_radius}"/>
+          <box size="${0.032+collision_radius} ${0.032+collision_radius} ${0.032+collision_radius}"/> <!--If collision radius parameter is positive, add .032 to account for origin-->
         </xacro:if>
       </geometry>
